File: pcb/_autosave-pcb.kicad_sch (KiCad schematic)
At the start: 23 parts, among them J1 Screw_Terminal_01x02, J2 Screw_Terminal_01x04, J3 Screw_Terminal_01x04, J4 Screw_Terminal_01x03, J5 Screw_Terminal_01x06, Q1 2N7000, Q2 2N7000, Q3 2N7000

Commit message: push rest
Parts:
- added MovingBumperStart1, MovingBumper_back1, MovingBumper_front1, Rehydration_bumper1: Screw_Terminal_01x03, TerminalBlock:TerminalBlock_MaiXu_MX126-5.0-03P_1x03_P5.00mm, symbol Connector:Screw_Terminal_01x03
- J2, J3: footprint (none) -> TerminalBlock:TerminalBlock_MaiXu_MX126-5.0-04P_1x04_P5.00mm
- J4: footprint (none) -> TerminalBlock:TerminalBlock_MaiXu_MX126-5.0-03P_1x03_P5.00mm
- J5: footprint (none) -> TerminalBlock:TerminalBlock_MaiXu_MX126-5.0-06P_1x06_P5.00mm
Connections:
- net at A1.1 (GND), A1.8 (VMOT), A2.1 (GND)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: now also Q1.1 (S), MovingBumperStart1.1 (Pin_1), MovingBumper_back1.1 (Pin_1), MovingBumper_front1.1 (Pin_1), Rehydration_bumper1.1 (Pin_1)
- net at Q2.3 (D): now also J5.3 (Pin_3)
- net at R2.1: now also ESP32-S3.19 (13)
- net at R2.2: now also Q1.2 (G)
- net at A1.13 (~{RST}), A1.14 (~{SLP}), A2.13 (~{RST})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: now also J5.2 (Pin_2), J5.4 (Pin_4), MovingBumperStart1.2 (Pin_2), MovingBumper_back1.2 (Pin_2), MovingBumper_front1.2 (Pin_2), Rehydration_bumper1.2 (Pin_2)
- net at R3.1: now also ESP32-S3.18 (12)
- net at ESP32-S3.13 (3): now also MovingBumper_front1.3 (Pin_3)
- net at ESP32-S3.15 (9): now also MovingBumperStart1.3 (Pin_3)
- net at ESP32-S3.16 (10): now also MovingBumper_back1.3 (Pin_3)
- net at ESP32-S3.34 (36): now also Rehydration_bumper1.3 (Pin_3)
- net at Q1.3 (D): now also J5.1 (Pin_1); no longer Q1.1 (S)
Other:
- moved on the sheet: Q1, R2
